File: M5stakATOM/Atomic/Atomic_V1.0__P-CAD-ASCII.Eagle-import-accel.ulp.brd (EAGLE design)
At the start: 76 parts

Commit message: small improvements
Other:
- board outline added: 20 x 44 mm
- board text added: "ToDo: - replace Pads for (error on the right outside of the board)"
