File: M5stakATOM/Atomic/Atomic_V1.0__P-CAD-ASCII.PCB.brd (EAGLE design)
At the start: 20 x 44 mm, 76 parts

Commit message: small improvements
Other:
- outline, holes or cut-outs redrawn
Changed lines of the file:
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@@
 <wire x1="-9.65" y1="33.4" x2="-8.35" y2="33.4" width="0.2" layer="20" curve="180"/>
 <wire x1="-8" y1="4.4" x2="-8" y2="11.6" width="0.2" layer="20" curve="180"/>
-<wire x1="1" y1="-6" x2="1" y2="-4" width="0.2" layer="21" curve="180"/>
-<wire x1="-1" y1="-4" x2="-1" y2="-6" width="0.2" layer="21" curve="180"/>
+<wire x1="1" y1="-6" x2="1" y2="-4" width="0.2" layer="20" curve="180"/>
+<wire x1="-1" y1="-4" x2="-1" y2="-6" width="0.2" layer="20" curve="180"/>
 <wire x1="-4.55" y1="33.5" x2="-3.45" y2="33.5" width="0.2" layer="20" curve="180"/>
 <wire x1="-1.4142125" y1="-9.4142125" x2="1.4142125" y2="-9.4142125" width="0.2" layer="20" curve="90"/>
 <wire x1="8.35" y1="33.4" x2="9.65" y2="33.4" width="0.2" layer="20" curve="180"/>
 <wire x1="3.45" y1="33.5" x2="4.55" y2="33.5" width="0.2" layer="20" curve="180"/>
-<circle x="-8" y="16" radius="1.6" width="0.2" layer="21"/>
-<circle x="8" y="16" radius="1.6" width="0.2" layer="21"/>
+<circle x="-8" y="16" radius="1.6" width="0.2" layer="20"/>
+<circle x="8" y="16" radius="1.6" width="0.2" layer="20"/>
 <wire x1="8" y1="11.6" x2="8" y2="4.4" width="0.2" layer="20" curve="180"/>
 <wire x1="0" y1="0" x2="0" y2="0.325" width="0" layer="21"/>
@@
 <wire x1="8.1" y1="34" x2="8.35" y2="33.75" width="0.2" layer="20"/>
 <wire x1="-10" y1="4.4" x2="-8" y2="4.4" width="0.2" layer="20"/>
-<wire x1="-1" y1="-6" x2="1" y2="-6" width="0.2" layer="21"/>
-<wire x1="-1" y1="-4" x2="1" y2="-4" width="0.2" layer="21"/>
+<wire x1="-1" y1="-6" x2="1" y2="-6" width="0.2" layer="20"/>
+<wire x1="-1" y1="-4" x2="1" y2="-4" width="0.2" layer="20"/>
 <wire x1="10" y1="-9.6" x2="10" y2="4.4" width="0.2" layer="20"/>
 <wire x1="9.6" y1="-10" x2="10" y2="-9.6" width="0.2" layer="20"/>
