File: M5stakATOM/Atomic/Atomic_V1.0__P-CAD-ASCII.PCB_DipTrace-Export.brd (EAGLE design)
At the start: 24 x 48.1 mm, 76 parts

Commit message: small improvements
Parts:
- removed FreePad0: FREEPAD, common:FreePad
- removed FreePad1, FreePad2, FreePad20, FreePad21, FreePad22, FreePad23, FreePad24, FreePad25, FreePad26, FreePad27, FreePad28, FreePad29, FreePad3, FreePad30, FreePad31, FreePad32, FreePad33, FreePad34, FreePad35, FreePad36, FreePad37, FreePad38, FreePad39, FreePad4, FreePad40, FreePad41, FreePad42, FreePad43, FreePad44, FreePad45, FreePad46, FreePad47, FreePad48, FreePad49, FreePad5, FreePad50, FreePad51, FreePad52, FreePad53, FreePad54, FreePad55, FreePad56, FreePad57, FreePad58, FreePad59, FreePad6, FreePad60, FreePad61, FreePad62, FreePad63, FreePad64, FreePad65, FreePad7, FreePad70, FreePad71, FreePad72, FreePad73, FreePad8, FreePad9: FREEPAD, common:FreePad_FreePad1
- removed FreePad10: FREEPAD, common:FreePad_FreePad10
- removed FreePad11, FreePad12, FreePad13, FreePad14, FreePad15, FreePad16, FreePad17, FreePad19: FREEPAD, common:FreePad_FreePad11
- removed FreePad18: FREEPAD, common:FreePad_FreePad18
- removed FreePad66: FREEPAD, common:FreePad_FreePad66
- removed FreePad67, FreePad68: FREEPAD, common:FreePad_FreePad67
- removed FreePad69: FREEPAD, common:FreePad_FreePad69
- removed FreePad74, FreePad75: FREEPAD, common:FreePad_FreePad74
- added FREEPAD0: FREEPAD, common:FREEPAD
- added FREEPAD1, FREEPAD2, FREEPAD20, FREEPAD21, FREEPAD22, FREEPAD23, FREEPAD24, FREEPAD25, FREEPAD26, FREEPAD27, FREEPAD28, FREEPAD29, FREEPAD3, FREEPAD30, FREEPAD31, FREEPAD32, FREEPAD33, FREEPAD34, FREEPAD35, FREEPAD36, FREEPAD37, FREEPAD38, FREEPAD39, FREEPAD4, FREEPAD40, FREEPAD41, FREEPAD42, FREEPAD43, FREEPAD44, FREEPAD45, FREEPAD46, FREEPAD47, FREEPAD48, FREEPAD49, FREEPAD5, FREEPAD50, FREEPAD51, FREEPAD52, FREEPAD53, FREEPAD54, FREEPAD55, FREEPAD56, FREEPAD57, FREEPAD58, FREEPAD59, FREEPAD6, FREEPAD60, FREEPAD61, FREEPAD62, FREEPAD63, FREEPAD64, FREEPAD65, FREEPAD7, FREEPAD70, FREEPAD71, FREEPAD72, FREEPAD73, FREEPAD8, FREEPAD9: FREEPAD, common:FREEPAD_FREEPAD1
- added FREEPAD10: FREEPAD, common:FREEPAD_FREEPAD10
- added FREEPAD11, FREEPAD12, FREEPAD13, FREEPAD14, FREEPAD15, FREEPAD16, FREEPAD17, FREEPAD19: FREEPAD, common:FREEPAD_FREEPAD11
- added FREEPAD18: FREEPAD, common:FREEPAD_FREEPAD18
- added FREEPAD66: FREEPAD, common:FREEPAD_FREEPAD66
- added FREEPAD67, FREEPAD68: FREEPAD, common:FREEPAD_FREEPAD67
- added FREEPAD69: FREEPAD, common:FREEPAD_FREEPAD69
- added FREEPAD74, FREEPAD75: FREEPAD, common:FREEPAD_FREEPAD74
Other:
- board size 24 x 48.1 mm -> 20 x 44 mm
