File: M5stakATOM/AtomHubProto/AtomHubProto-P-CAD-ACCEL-ascii.DiptraceExport.PCB.eagle.brd (EAGLE design)
At the start: 36 x 68 mm, 304 parts

Commit message: add template: atom-hub-proto-self-Vorlage.xxx
Parts:
- removed GROVE: GPIO_Socket_4P, common:GROVE
- added E$1: (no value), common:GROVE-NEU
Connections:
- net 5V: no longer GROVE.4
- net GND: no longer GROVE.3
